File: PCB/Orcus/Orcus.kicad_pcb (KiCad board)
At the start: 2 copper layers, 258.2 x 87.7 mm, 84 parts, among them J1 -, J2 -, J3 +, J4 +, J5 LED, J6 LED, SW1 MX_LED, SW10 MX_LED, SW11 MX_LED, SW12 MX_LED, SW13 MX_LED, SW14 MX_LED, SW15 MX_LED, SW16 MX_LED, SW17 MX_LED, SW18 MX_LED, SW19 MX_LED, SW2 MX_LED, SW20 MX_LED, SW21 MX_LED, SW22 MX_LED, SW23 MX_LED, SW24 MX_LED, SW25 MX_LED, SW26 MX_LED, SW27 MX_LED, SW28 MX_LED, SW29 MX_LED, SW3 MX_LED, SW30 MX_LED, SW31 MX_LED, SW32 MX_LED, SW33 MX_LED, SW34 MX_LED, SW35 MX_LED, SW36 MX_LED, SW37 MX_LED, SW38 MX_LED, SW4 MX_LED, SW5 MX_LED, SW6 MX_LED, SW7 MX_LED, SW8 MX_LED, SW9 MX_LED, U1 XIAO-nRF52840-SMD, U3 XIAO-nRF52840-SMD

Commit message: almost final
Routing:
- net col1-1: track 0.00 -> 194.9 mm
- net col2-1: track 0.00 -> 160.4 mm
- net row3-1: track 0.00 -> 152.7 mm
- net col0-1: track 0.00 -> 152.4 mm
- net row3: track 14.7 -> 144.5 mm
- net row2-1: track 0.00 -> 127.1 mm
- net row1-1: track 0.00 -> 115.7 mm
- net Gnd-1: track 0.00 -> 113.4 mm
- net Net-(J4-Pin_1): track 0.00 -> 105.7 mm
- net 5v-1: track 0.00 -> 102.7 mm, vias 0 -> 2
- net row0-1: track 0.00 -> 102.2 mm
- net Net-(J2-Pin_1): track 0.00 -> 102.1 mm
- net Data-1: track 0.00 -> 92.8 mm
- net row0: track 33.9 -> 126.5 mm
- net row1: track 34.2 -> 126.2 mm
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