File: PCB/Orcus/Orcus.kicad_sch (KiCad schematic)
At the start: 78 parts, among them SW1 MX_LED, SW10 MX_LED, SW11 MX_LED, SW12 MX_LED, SW13 MX_LED, SW14 MX_LED, SW15 MX_LED, SW16 MX_LED, SW17 MX_LED, SW18 MX_LED, SW19 MX_LED, SW2 MX_LED, SW20 MX_LED, SW21 MX_LED, SW22 MX_LED, SW23 MX_LED, SW24 MX_LED, SW25 MX_LED, SW26 MX_LED, SW27 MX_LED, SW28 MX_LED, SW29 MX_LED, SW3 MX_LED, SW30 MX_LED, SW31 MX_LED, SW32 MX_LED, SW33 MX_LED, SW34 MX_LED, SW35 MX_LED, SW36 MX_LED, SW37 MX_LED, SW38 MX_LED, SW4 MX_LED, SW5 MX_LED, SW6 MX_LED, SW7 MX_LED, SW8 MX_LED, SW9 MX_LED, U1 SeeeduinoXIAO, U2 SeeeduinoXIAO

Commit message: update footprint, remove traces
Parts:
- D1, D10, D11, D12, D13, D14, D15, D16, D17, D18, D19, D2, D20, D21, D22, D23, D24, D25, D26, D27, D28, D29, D3, D30, D31, D32, D33, D34, D35, D36, D37, D38, D4, D5, D6, D7, D8, D9: footprint Keebio-Parts.pretty-master:D_SOD123-Hole -> Keebio-Parts.pretty-master:D_SOD123F-Hole
- U1, U2: footprint Seeeduino XIAO KICAD:Seeeduino XIAO-MOUDLE14P-2.54-21X17.8MM -> Seeeduino XIAO KICAD:Seeeduino XIAO-MOUDLE14P-2.54-21X17.8MM-holes
Changed lines of the file:
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@@
 			)
 		)
-		(property "Footprint" "Keebio-Parts.pretty-master:D_SOD123-Hole"
+		(property "Footprint" "Keebio-Parts.pretty-master:D_SOD123F-Hole"
 			(at 77.47 185.42 0)
 			(effects
@@
 			)
 		)
-		(property "Footprint" "Keebio-Parts.pretty-master:D_SOD123-Hole"
+		(property "Footprint" "Keebio-Parts.pretty-master:D_SOD123F-Hole"
 			(at 152.4 95.25 0)
 			(effects
@@
 			)
 		)
-		(property "Footprint" "Keebio-Parts.pretty-master:D_SOD123-Hole"
+		(property "Footprint" "Keebio-Parts.pretty-master:D_SOD123F-Hole"
 			(at 97.79 39.37 0)
 			(effects
@@
 			)
 		)
-		(property "Footprint" "Keebio-Parts.pretty-master:D_SOD123-Hole"
+		(property "Footprint" "Keebio-Parts.pretty-master:D_SOD123F-Hole"
 			(at 116.84 57.15 0)
 			(effects
@@
 			)
 		)
-		(property "Footprint" "Keebio-Parts.pretty-master:D_SOD123-Hole"
+		(property "Footprint" "Keebio-Parts.pretty-master:D_SOD123F-Hole"
 			(at 58.42 76.2 0)
 			(effects
@@
 			)
 		)
-		(property "Footprint" "Keebio-Parts.pretty-master:D_SOD123-Hole"
+		(property "Footprint" "Keebio-Parts.pretty-master:D_SOD123F-Hole"
 			(at 118.11 128.27 0)
 			(effects
@@
 			)
 		)
-		(property "Footprint" "Keebio-Parts.pretty-master:D_SOD123-Hole"
+		(property "Footprint" "Keebio-Parts.pretty-master:D_SOD123F-Hole"
 			(at 116.84 39.37 0)
 			(effects
@@
 			)
 		)
-		(property "Footprint" "Keebio-Parts.pretty-master:D_SOD123-Hole"
+		(property "Footprint" "Keebio-Parts.pretty-master:D_SOD123F-Hole"
 			(at 58.42 39.37 0)
 			(effects
@@
 			)
 		)
-		(property "Footprint" "Keebio-Parts.pretty-master:D_SOD123-Hole"
+		(property "Footprint" "Keebio-Parts.pretty-master:D_SOD123F-Hole"
 			(at 134.62 76.2 0)
 			(effects
@@
 			)
 		)
-		(property "Footprint" "Keebio-Parts.pretty-master:D_SOD123-Hole"
+		(property "Footprint" "Keebio-Parts.pretty-master:D_SOD123F-Hole"
 			(at 41.91 185.42 0)
 			(effects
@@
 			)
 		)
-		(property "Footprint" "Keebio-Parts.pretty-master:D_SOD123-Hole"
+		(property "Footprint" "Keebio-Parts.pretty-master:D_SOD123F-Hole"
 			(at 99.06 165.1 0)
 			(effects
@@
 			)
 		)
-		(property "Footprint" "Keebio-Parts.pretty-master:D_SOD123-Hole"
+		(property "Footprint" "Keebio-Parts.pretty-master:D_SOD123F-Hole"
 			(at 59.69 185.42 0)
 			(effects
@@
 			)
 		)
-		(property "Footprint" "Keebio-Parts.pretty-master:D_SOD123-Hole"
+		(property "Footprint" "Keebio-Parts.pretty-master:D_SOD123F-Hole"
 			(at 58.42 57.15 0)
 			(effects
@@
 			)
 		)
-		(property "Footprint" "Keebio-Parts.pretty-master:D_SOD123-Hole"
+		(property "Footprint" "Keebio-Parts.pretty-master:D_SOD123F-Hole"
 			(at 97.79 57.15 0)
 			(effects
@@
 			)
 		)
-		(property "Footprint" "Keebio-Parts.pretty-master:D_SOD123-Hole"
+		(property "Footprint" "Keebio-Parts.pretty-master:D_SOD123F-Hole"
 			(at 78.74 39.37 0)
 			(effects
@@
 			)
 		)
-		(property "Footprint" "Keebio-Parts.pretty-master:D_SOD123-Hole"
+		(property "Footprint" "Keebio-Parts.pretty-master:D_SOD123F-Hole"
 			(at 80.01 165.1 0)
 			(effects
@@
 			)
 		)
-		(property "Footprint" "Keebio-Parts.pretty-master:D_SOD123-Hole"
+		(property "Footprint" "Keebio-Parts.pretty-master:D_SOD123F-Hole"
 			(at 36.83 57.15 0)
 			(effects
@@
 			)
 		)
-		(property "Footprint" "Keebio-Parts.pretty-master:D_SOD123-Hole"
+		(property "Footprint" "Keebio-Parts.pretty-master:D_SOD123F-Hole"
 			(at 59.69 128.27 0)
 			(effects
@@
 			)
 		)
-		(property "Footprint" "Keebio-Parts.pretty-master:D_SOD123-Hole"
+		(property "Footprint" "Keebio-Parts.pretty-master:D_SOD123F-Hole"
 			(at 134.62 39.37 0)
 			(effects
@@
 			)
 		)
-		(property "Footprint" "Keebio-Parts.pretty-master:D_SOD123-Hole"
+		(property "Footprint" "Keebio-Parts.pretty-master:D_SOD123F-Hole"
 			(at 116.84 76.2 0)
 			(effects
@@
 			)
 		)
-		(property "Footprint" "Keebio-Parts.pretty-master:D_SOD123-Hole"
+		(property "Footprint" "Keebio-Parts.pretty-master:D_SOD123F-Hole"
 			(at 78.74 57.15 0)
 			(effects
@@
 			)
 		)
-		(property "Footprint" "Keebio-Parts.pretty-master:D_SOD123-Hole"
+		(property "Footprint" "Keebio-Parts.pretty-master:D_SOD123F-Hole"
 			(at 156.21 146.05 0)
 			(effects
@@
 			)
 		)
-		(property "Footprint" "Keebio-Parts.pretty-master:D_SOD123-Hole"
+		(property "Footprint" "Keebio-Parts.pretty-master:D_SOD123F-Hole"
 			(at 99.06 146.05 0)
 			(effects
@@
 			)
 		)
-		(property "Footprint" "Keebio-Parts.pretty-master:D_SOD123-Hole"
+		(property "Footprint" "Keebio-Parts.pretty-master:D_SOD123F-Hole"
 			(at 99.06 128.27 0)
 			(effects
@@
 			)
 		)
-		(property "Footprint" "Keebio-Parts.pretty-master:D_SOD123-Hole"
+		(property "Footprint" "Keebio-Parts.pretty-master:D_SOD123F-Hole"
 			(at 59.69 165.1 0)
 			(effects
@@
 			)
 		)
-		(property "Footprint" "Keebio-Parts.pretty-master:D_SOD123-Hole"
+		(property "Footprint" "Keebio-Parts.pretty-master:D_SOD123F-Hole"
 			(at 118.11 146.05 0)
 			(effects
@@
 			)
 		)
-		(property "Footprint" "Keebio-Parts.pretty-master:D_SOD123-Hole"
+		(property "Footprint" "Keebio-Parts.pretty-master:D_SOD123F-Hole"
 			(at 97.79 76.2 0)
 			(effects
@@
 			)
 		)
-		(property "Footprint" "Keebio-Parts.pretty-master:D_SOD123-Hole"
+		(property "Footprint" "Keebio-Parts.pretty-master:D_SOD123F-Hole"
 			(at 135.89 128.27 0)
 			(effects
@@
 			)
 		)
-		(property "Footprint" "Keebio-Parts.pretty-master:D_SOD123-Hole"
+		(property "Footprint" "Keebio-Parts.pretty-master:D_SOD123F-Hole"
 			(at 116.84 95.25 0)
 			(effects
@@
 			)
 		)
-		(property "Footprint" "Keebio-Parts.pretty-master:D_SOD123-Hole"
+		(property "Footprint" "Keebio-Parts.pretty-master:D_SOD123F-Hole"
 			(at 118.11 165.1 0)
 			(effects
@@
 			)
 		)
-		(property "Footprint" "Keebio-Parts.pretty-master:D_SOD123-Hole"
+		(property "Footprint" "Keebio-Parts.pretty-master:D_SOD123F-Hole"
 			(at 134.62 57.15 0)
 			(effects
@@
 			)
 		)
-		(property "Footprint" "Keebio-Parts.pretty-master:D_SOD123-Hole"
+		(property "Footprint" "Keebio-Parts.pretty-master:D_SOD123F-Hole"
 			(at 134.62 95.25 0)
 			(effects
@@
 			)
 		)
-		(property "Footprint" "Keebio-Parts.pretty-master:D_SOD123-Hole"
+		(property "Footprint" "Keebio-Parts.pretty-master:D_SOD123F-Hole"
 			(at 135.89 146.05 0)
 			(effects
@@
 			)
 		)
-		(property "Footprint" "Keebio-Parts.pretty-master:D_SOD123-Hole"
+		(property "Footprint" "Keebio-Parts.pretty-master:D_SOD123F-Hole"
 			(at 135.89 165.1 0)
 			(effects
@@
 			)
 		)
-		(property "Footprint" "Keebio-Parts.pretty-master:D_SOD123-Hole"
+		(property "Footprint" "Keebio-Parts.pretty-master:D_SOD123F-Hole"
 			(at 78.74 76.2 0)
 			(effects
@@
 			)
 		)
-		(property "Footprint" "Keebio-Parts.pretty-master:D_SOD123-Hole"
+		(property "Footprint" "Keebio-Parts.pretty-master:D_SOD123F-Hole"
 			(at 80.01 128.27 0)
 			(effects
@@
 			)
 		)
-		(property "Footprint" "Keebio-Parts.pretty-master:D_SOD123-Hole"
+		(property "Footprint" "Keebio-Parts.pretty-master:D_SOD123F-Hole"
 			(at 80.01 146.05 0)
 			(effects
@@
 			)
 		)
-		(property "Footprint" "Seeeduino XIAO KICAD:Seeeduino XIAO-MOUDLE14P-2.54-21X17.8MM"
+		(property "Footprint" "Seeeduino XIAO KICAD:Seeeduino XIAO-MOUDLE14P-2.54-21X17.8MM-holes"
 			(at 222.25 130.81 0)
 			(effects
@@
 			)
 		)
-		(property "Footprint" "Seeeduino XIAO KICAD:Seeeduino XIAO-MOUDLE14P-2.54-21X17.8MM"
+		(property "Footprint" "Seeeduino XIAO KICAD:Seeeduino XIAO-MOUDLE14P-2.54-21X17.8MM-holes"
 			(at 220.98 49.53 0)
 			(effects
@@
 			)
 		)
-		(property "Footprint" "Keebio-Parts.pretty-master:D_SOD123-Hole"
+		(property "Footprint" "Keebio-Parts.pretty-master:D_SOD123F-Hole"
 			(at 59.69 146.05 0)
 			(effects

Commit message: traces remaining
Parts:
- removed U1, U2: SeeeduinoXIAO, Seeeduino XIAO KICAD:Seeeduino XIAO-MOUDLE14P-2.54-21X17.8MM-holes, symbol Seeeduino XIAO:SeeeduinoXIAO
- added J1, J2: -, TOTEMlib:BatteryPad, symbol Connector:Conn_01x01_Pin
- added J3, J4: +, TOTEMlib:BatteryPad, symbol Connector:Conn_01x01_Pin
- added J5, J6: LED, Keebio-Parts.pretty-master:NeoPixel_Mini_Button-v2, symbol Connector:Conn_01x03_Pin
- added U1, U3: XIAO-nRF52840-SMD, TOTEMlib:xiao-ble-smd-cutout-mod, symbol MCU_SEEED_XIAO_Series:XIAO-nRF52840-SMD
Connections:
- net col0: now also U3.7 (PB08_A6_D6_TX)
- net col0-1: now also U1.7 (PB08_A6_D6_TX)
- net col1: now also U3.8 (PB09_A7_D7_RX)
- net col1-1: now also U1.8 (PB09_A7_D7_RX)
- net col2: now also U3.9 (PA7_A8_D8_SCK)
- net col2-1: now also U1.9 (PA7_A8_D8_SCK)
- net col3: now also U3.10 (PA5_A9_D9_MISO)
- net col3-1: now also U1.10 (PA5_A9_D9_MISO)
- net col4: now also U3.11 (PA6_A10_D10_MOSI)
- net col4-1: now also U1.11 (PA6_A10_D10_MOSI)
- net row0: now also U3.3 (PA10_A2_D2)
- net row0-1: now also U1.3 (PA10_A2_D2)
- net row1: now also U3.4 (PA11_A3_D3)
- net row1-1: now also U1.4 (PA11_A3_D3)
- net row2: now also U3.5 (PA8_A4_D4_SDA)
- net row2-1: now also U1.5 (PA8_A4_D4_SDA)
- net row3: now also U3.6 (PA9_A5_D5_SCL)
- net row3-1: now also U1.6 (PA9_A5_D5_SCL)
- new net: J4.1 (Pin_1), U1.15 (BAT)
- new net: J2.1 (Pin_1), U1.16 (GND)
- new net: J1.1 (Pin_1), U3.16 (GND)
- new net: J3.1 (Pin_1), U3.15 (BAT)
- new net 5v: J5.1 (Pin_1), U3.14 (5V)
- new net 5v-1: J6.1 (Pin_1), U1.14 (5V)
- new net Data: J5.2 (Pin_2), U3.2 (PA4_A1_D1)
- new net Data-1: J6.2 (Pin_2), U1.2 (PA4_A1_D1)
- new net Gnd: J5.3 (Pin_3), U3.13 (GND)
- new net Gnd-1: J6.3 (Pin_3), U1.13 (GND)

Commit message: replaced pad
Parts:
- J1, J2, J3, J4: footprint TOTEMlib:BatteryPad -> Keebio-Parts.pretty-master:Wire_Pad_24AWG
Changed lines of the file:
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@@
 			)
 		)
-		(property "Footprint" "TOTEMlib:BatteryPad"
+		(property "Footprint" "Keebio-Parts.pretty-master:Wire_Pad_24AWG"
 			(at 222.25 85.09 0)
 			(effects
@@
 			)
 		)
-		(property "Footprint" "TOTEMlib:BatteryPad"
+		(property "Footprint" "Keebio-Parts.pretty-master:Wire_Pad_24AWG"
 			(at 218.44 158.75 0)
 			(effects
@@
 			)
 		)
-		(property "Footprint" "TOTEMlib:BatteryPad"
+		(property "Footprint" "Keebio-Parts.pretty-master:Wire_Pad_24AWG"
 			(at 218.44 85.09 0)
 			(effects
@@
 			)
 		)
-		(property "Footprint" "TOTEMlib:BatteryPad"
+		(property "Footprint" "Keebio-Parts.pretty-master:Wire_Pad_24AWG"
 			(at 222.25 158.75 0)
 			(effects

Commit message: updated pcb and sch
Parts:
- D1, D10, D11, D12, D13, D14, D15, D16, D17, D18, D19, D2, D20, D21, D22, D23, D24, D25, D26, D27, D28, D29, D3, D30, D31, D32, D33, D34, D35, D36, D37, D38, D4, D5, D6, D7, D8, D9: footprint Keebio-Parts.pretty-master:D_SOD123F-Hole -> Keebio-Parts.pretty-master:D_SOD123F
Connections:
- net Data: now also U3.11 (PA6_A10_D10_MOSI); no longer U3.2 (PA4_A1_D1)
- net Data-1: now also U1.11 (PA6_A10_D10_MOSI); no longer U1.2 (PA4_A1_D1)
- net col1: now also U3.6 (PA9_A5_D5_SCL); no longer U3.8 (PB09_A7_D7_RX)
- net col1-1: now also U1.6 (PA9_A5_D5_SCL); no longer U1.8 (PB09_A7_D7_RX)
- net col2: now also U3.5 (PA8_A4_D4_SDA); no longer U3.9 (PA7_A8_D8_SCK)
- net col2-1: now also U1.5 (PA8_A4_D4_SDA); no longer U1.9 (PA7_A8_D8_SCK)
- net col3: now also U3.8 (PB09_A7_D7_RX); no longer U3.10 (PA5_A9_D9_MISO)
- net col3-1: now also U1.8 (PB09_A7_D7_RX); no longer U1.10 (PA5_A9_D9_MISO)
- net col4: now also U3.9 (PA7_A8_D8_SCK); no longer U3.11 (PA6_A10_D10_MOSI)
- net col4-1: now also U1.9 (PA7_A8_D8_SCK); no longer U1.11 (PA6_A10_D10_MOSI)
- net row0: now also U3.1 (PA02_A0_D0); no longer U3.3 (PA10_A2_D2)
- net row0-1: now also U1.1 (PA02_A0_D0); no longer U1.3 (PA10_A2_D2)
- net row1: now also U3.2 (PA4_A1_D1); no longer U3.4 (PA11_A3_D3)
- net row1-1: now also U1.2 (PA4_A1_D1); no longer U1.4 (PA11_A3_D3)
- net row2: now also U3.3 (PA10_A2_D2); no longer U3.5 (PA8_A4_D4_SDA)
- net row2-1: now also U1.3 (PA10_A2_D2); no longer U1.5 (PA8_A4_D4_SDA)
- net row3: now also U3.4 (PA11_A3_D3); no longer U3.6 (PA9_A5_D5_SCL)
- net row3-1: now also U1.4 (PA11_A3_D3); no longer U1.6 (PA9_A5_D5_SCL)

Commit message: new sch
Parts:
- removed J1, J2: -, Keebio-Parts.pretty-master:Wire_Pad_24AWG, symbol Connector:Conn_01x01_Pin
- removed J3, J4: +, Keebio-Parts.pretty-master:Wire_Pad_24AWG, symbol Connector:Conn_01x01_Pin
- removed J5, J6: LED, Keebio-Parts.pretty-master:NeoPixel_Mini_Button-v2, symbol Connector:Conn_01x03_Pin
- removed U1, U3: XIAO-nRF52840-SMD, TOTEMlib:xiao-ble-smd-cutout-mod, symbol MCU_SEEED_XIAO_Series:XIAO-nRF52840-SMD
- added SW39, SW40: MX_LED, Keebio-Parts.pretty-master:Kailh-PG1350-1u-NoLED, symbol keebio:MX_LED
- added U1, U2: XIAO-nRF52840-DIP, MCU_SEEED_XIAO_Series:XIAO-nRF52840-DIP, symbol MCU_SEEED_XIAO_Series:XIAO-nRF52840-DIP
Connections:
- net col0 renamed L-col0
- net L-col0: now also U2.7 (PB08_A6_D6_TX)
- net col0-1 renamed R-col0
- net R-col0: now also U1.7 (PB08_A6_D6_TX)
- net col1 renamed L-col1
- net L-col1: now also U2.6 (PA9_A5_D5_SCL)
- net col1-1 renamed R-col1
- net R-col1: now also U1.6 (PA9_A5_D5_SCL)
- net col2 renamed L-col2
- net L-col2: now also U2.5 (PA8_A4_D4_SDA)
- net col2-1 renamed R-col2
- net R-col2: now also U1.5 (PA8_A4_D4_SDA)
- net col3 renamed L-col3
- net L-col3: now also U2.8 (PB09_A7_D7_RX)
- net col3-1 renamed R-col3
- net R-col3: now also U1.8 (PB09_A7_D7_RX)
- net col4 renamed L-col4
- net L-col4: now also U2.9 (PA7_A8_D8_SCK)
- net col4-1 renamed R-col4
- net R-col4: now also U1.9 (PA7_A8_D8_SCK)
- net row0 renamed L-row0
- net L-row0: now also U2.1 (PA02_A0_D0)
- net row0-1 renamed R-row0
- net R-row0: now also U1.1 (PA02_A0_D0)
- net row1 renamed L-row1
- net L-row1: now also U2.2 (PA4_A1_D1)
- net row1-1 renamed R-row1
- net R-row1: now also U1.2 (PA4_A1_D1)
- net row2 renamed L-row2
- net L-row2: now also U2.3 (PA10_A2_D2)
- net row2-1 renamed R-row2
- net R-row2: now also U1.3 (PA10_A2_D2)
- net row3 renamed L-row3
- net L-row3: now also U2.4 (PA11_A3_D3)
- net row3-1 renamed R-row3
- net R-row3: now also U1.4 (PA11_A3_D3)
Other:
- moved on the sheet: D1, D10, D11, D12, D13, D14, D15, D16, D17, D18, D19, D2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

Commit message: updated pcb
Parts:
- U1: renamed from U2; footprint MCU_SEEED_XIAO_Series:XIAO-nRF52840-DIP -> SeeedStudio_XIAO_nRF52840_v1.1_KiCAD:XIAO-nRF52840-DIP
- U2: renamed from U1; footprint MCU_SEEED_XIAO_Series:XIAO-nRF52840-DIP -> SeeedStudio_XIAO_nRF52840_v1.1_KiCAD:XIAO-nRF52840-DIP
- renumbered D11 to D10, D12 to D11, D13 to D12, D14 to D13, D15 to D14, D16 to D15, D6 to D16, D31 to D30, D32 to D31, D33 to D32, D34 to D33, D35 to D34, D36 to D35, D37 to D36, D38 to D37, D30 to D38, D7 to D6, D8 to D7, D9 to D8, D10 to D9, SW11 to SW10, SW12 to SW11, SW13 to SW12, SW14 to SW13, SW15 to SW14, SW16 to SW15, SW6 to SW16, SW31 to SW30, SW32 to SW31, SW33 to SW32, SW34 to SW33, SW35 to SW34, SW36 to SW35, SW37 to SW36, SW38 to SW37, SW30 to SW38, SW7 to SW6, SW8 to SW7, SW9 to SW8, SW10 to SW9
Connections:
- no-connect marks 0 -> 10
