File: PCB/Orcus/Orcus.kicad_sch (KiCad schematic)
At the start: 80 parts, among them SW1 MX_LED, SW10 MX_LED, SW11 MX_LED, SW12 MX_LED, SW13 MX_LED, SW14 MX_LED, SW15 MX_LED, SW16 MX_LED, SW17 MX_LED, SW18 MX_LED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

Commit message: sch update
Parts:
- added SW41, SW42, SW43, SW44: BATT, Keebio-Parts.pretty-master:Reset_Breakout, symbol keebio:MX_LED
- SW39, SW40: value MX_LED -> RESET
Connections:
- new net: SW41.1, SW42.1
- new net: SW41.2, SW42.2
- new net: SW43.1, SW44.1
- new net: SW43.2, SW44.2
